File: pcb/serial-logger-prototype.sch (KiCad schematic (older format))
At the start: 69 parts, among them J1 Conn_ARM_JTAG_SWD_10, J2 Conn_01x04_Female, J3 Conn_01x04_Female, J4 Conn_01x03_Male, SW1 Rotary_Encoder_Switch_DualLED, SW2 SW_SPDT, U1 STM32G070KBT6, U2 74LVC3G17, U3 TLV70228_SOT23-5, U4 sn74lv1t34, U5 TLV61046ADB, U6 sn74lv1t34

Commit message: Add Final production BOM
Parts:
- BT1: Alt (none) -> 1043; MPN (none) -> 1043P; Mouser (none) -> 534-1043P
- H1: MPN (none) -> ELW2106AA; Mouser (none) -> 387-ELW2106AA
- H2, H3, H4: value MountingHole_Pad -> DNI
- J1: value Conn_ARM_JTAG_SWD_10 -> JTAG/SWD; Alt (none) -> FTSH-105-01-L-DV (cheaper, no fancy shroud); Farnell (none) -> 2856437; MPN (none) -> FTSH-105-01-L-DV-K-P; Mouser (none) -> 200-FTSH10501LDVKP
- J2: Farnell (none) -> 1593460
- J3: value Conn_01x04_Female -> Conn_01x04_Male; Farnell (none) -> 2888929
- MB1, MB2, MB3, MB4: value MouseBite -> DNI
- SW1: Alternative (none) -> PEL12D-4225S-S1024 (blue/orange LEDS); MPN (none) -> PEL12D-4225S-S2024; Mouser (none) -> 652-PEL12D4225SS2024
- SW2: Farnell (none) -> 1608080; MPN (none) -> 09.03201.02
- TH1, TH2, TH3, TH4: value ToolingHole -> DNI
- U1: Farnell (none) -> 3365394; MPN (none) -> STM32G070KBT6; Mouser (none) -> 511-STM32G070KBT6
- U2: Farnell (none) -> 1236391; MPN (none) -> SN74LVC3G17DCT
- U3: Farnell (none) -> 2492371; MPN (none) -> TLV70228DBVT
- U4, U6: Farnell (none) -> 3119564; MPN (none) -> SN74LV1T34DBVR; Mouser (none) -> 595-SN74LV1T34DBVR
- U5: Farnell (none) -> 3007283; MPN (none) -> TLV61046ADBV
Other:
- note added: "TODO all 10k resistors\nsame footprint!"
Changed lines of the file:
@@
 F 2 "Jitter_Footprints:Molex_503480-1400-1x14-1MP_P0.5mm_Horizontal" H 14200 3350 50  0001 C CNN
 F 3 "https://nl.mouser.com/datasheet/2/921/Futaba-10-02-2018-ELW2106AA_A_03_SHORT-1487521.pdf" H 14200 3350 50  0001 C CNN
+F 4 "ELW2106AA" H 14200 3350 50  0001 C CNN "MPN"
+F 5 "387-ELW2106AA" H 14200 3350 50  0001 C CNN "Mouser"
 	1    14200 3350
 	1    0    0    -1
@@
 F 2 "Jitter_Footprints:BatteryHolder_Keystone_1043(p)_1x18650" V 950 7660 50  0001 C CNN
 F 3 "~" V 950 7660 50  0001 C CNN
+F 4 "1043P" H 950 7600 50  0001 C CNN "MPN"
+F 5 "534-1043P" H 950 7600 50  0001 C CNN "Mouser"
+F 6 "1043" H 950 7600 50  0001 C CNN "Alt"
 	1    950  7600
 	1    0    0    -1
@@
 P 6850 3800
 F 0 "J1" H 6407 3846 50  0000 R CNN
-F 1 "Conn_ARM_JTAG_SWD_10" H 7150 2800 50  0000 R CNN
+F 1 "JTAG/SWD" H 7150 2800 50  0000 R CNN
 F 2 "Connector_PinHeader_1.27mm:PinHeader_2x05_P1.27mm_Vertical_SMD" H 6850 3800 50  0001 C CNN
 F 3 "http://infocenter.arm.com/help/topic/com.arm.doc.ddi0314h/DDI0314H_coresight_components_trm.pdf" V 6500 2550 50  0001 C CNN
+F 4 "FTSH-105-01-L-DV-K-P" H 6850 3800 50  0001 C CNN "MPN"
+F 5 "FTSH-105-01-L-DV (cheaper, no fancy shroud)" H 6850 3800 50  0001 C CNN "Alt"
+F 6 "2856437" H 6850 3800 50  0001 C CNN "Farnell"
+F 7 "200-FTSH10501LDVKP" H 6850 3800 50  0001 C CNN "Mouser"
 	1    6850 3800
 	1    0    0    -1
@@
 P 5350 8200
 F 0 "J3" H 5242 8485 50  0000 C CNN
-F 1 "Conn_01x04_Female" H 5242 8394 50  0000 C CNN
+F 1 "Conn_01x04_Male" H 5242 8394 50  0001 C CNN
 F 2 "Connector_PinHeader_2.54mm:PinHeader_1x04_P2.54mm_Horizontal" H 5350 8200 50  0001 C CNN
 F 3 "~" H 5350 8200 50  0001 C CNN
+F 4 "2888929" H 5350 8200 50  0001 C CNN "Farnell"
 	1    5350 8200
 	-1   0    0    -1
@@
 F 2 "Package_TO_SOT_SMD:SOT-23-5" H 7200 8000 50  0001 C CNN
 F 3 "http://www.ti.com/lit/ds/symlink/sn74lv1t34.pdf" H 7200 8000 50  0001 C CNN
+F 4 "SN74LV1T34DBVR" H 7250 7900 50  0001 C CNN "MPN"
+F 5 "595-SN74LV1T34DBVR" H 7250 7900 50  0001 C CNN "Mouser"
+F 6 "3119564" H 7250 7900 50  0001 C CNN "Farnell"
 	1    7250 7900
 	-1   0    0    -1
@@
 F 2 "Package_TO_SOT_SMD:SOT-23-5" H 6950 9200 50  0001 C CNN
 F 3 "http://www.ti.com/lit/ds/symlink/sn74lv1t34.pdf" H 6950 9200 50  0001 C CNN
+F 4 "SN74LV1T34DBVR" H 7000 9100 50  0001 C CNN "MPN"
+F 5 "595-SN74LV1T34DBVR" H 7000 9100 50  0001 C CNN "Mouser"
+F 6 "3119564" H 7000 9100 50  0001 C CNN "Farnell"
 	1    7000 9100
 	1    0    0    -1
@@
 F 3 "https://www.st.com/resource/en/datasheet/stm32g070kb.pdf" H 9450 2850 50  0001 C CNN
 F 4 "https://www.st.com/content/ccc/resource/technical/document/reference_manual/group0/fd/a3/20/58/ac/b0/48/23/DM00463896/files/DM00463896.pdf/jcr:content/translations/en.DM00463896.pdf" H 9150 2850 50  0001 C CNN "Manual"
+F 5 "STM32G070KBT6" H 9300 2850 50  0001 C CNN "MPN"
+F 6 "3365394" H 9300 2850 50  0001 C CNN "Farnell"
+F 7 "511-STM32G070KBT6" H 9300 2850 50  0001 C CNN "Mouser"
 	1    9300 2850
 	1    0    0    -1
@@
 F 2 "Package_SO:TSSOP-8_3x3mm_P0.65mm" H 3200 4900 50  0001 C CNN
 F 3 "http://www.ti.com/lit/sg/scyt129e/scyt129e.pdf" H 3200 4900 50  0001 C CNN
+F 4 "SN74LVC3G17DCT" H 3200 4900 50  0001 C CNN "MPN"
+F 5 "1236391" H 3200 4900 50  0001 C CNN "Farnell"
 	2    3200 4900
 	1    0    0    -1
@@
 F 2 "Package_SO:TSSOP-8_3x3mm_P0.65mm" H 3200 4150 50  0001 C CNN
 F 3 "http://www.ti.com/lit/sg/scyt129e/scyt129e.pdf" H 3200 4150 50  0001 C CNN
+F 4 "SN74LVC3G17DCT" H 3200 4150 50  0001 C CNN "MPN"
+F 5 "1236391" H 3200 4150 50  0001 C CNN "Farnell"
 	1    3200 4150
 	1    0    0    -1
@@
 F 2 "Package_TO_SOT_SMD:SOT-23-5" H 3250 7875 50  0001 C CIN
 F 3 "http://www.ti.com/lit/ds/symlink/tlv702.pdf" H 3250 7600 50  0001 C CNN
+F 4 "TLV70228DBVT" H 3250 7550 50  0001 C CNN "MPN"
+F 5 "2492371" H 3250 7550 50  0001 C CNN "Farnell"
 	1    3250 7550
 	1    0    0    -1
@@
 F 2 "Jitter_Footprints:PEL12D-4xxxS-Sxxxx" H 2150 2400 50  0001 C CNN
 F 3 "https://nl.mouser.com/datasheet/2/54/PEL12D-777459.pdf" H 2150 2210 50  0001 C CNN
+F 4 "PEL12D-4225S-S2024" H 2150 1950 50  0001 C CNN "MPN"
+F 5 "652-PEL12D4225SS2024" H 2150 1950 50  0001 C CNN "Mouser"
+F 6 "PEL12D-4225S-S1024 (blue/orange LEDS)" H 2150 1950 50  0001 C CNN "Alternative"
 	1    2150 1950
 	1    0    0    -1
@@
 F 2 "Jitter_Footprints:slide_switch_09.03201.02" H 1500 7450 50  0001 C CNN
 F 3 "~" H 1500 7450 50  0001 C CNN
+F 4 "09.03201.02" H 1500 7450 50  0001 C CNN "MPN"
+F 5 "1608080" H 1500 7450 50  0001 C CNN "Farnell"
 	1    1500 7450
 	-1   0    0    -1
@@
 P 9950 9300
 F 0 "H2" H 10050 9349 50  0000 L CNN
-F 1 "MountingHole_Pad" H 10050 9258 50  0000 L CNN
+F 1 "DNI" H 10050 9258 50  0001 L CNN
 F 2 "MountingHole:MountingHole_2.2mm_M2_Pad_Via" H 9950 9300 50  0001 C CNN
 F 3 "~" H 9950 9300 50  0001 C CNN
@@
 P 9950 9850
 F 0 "H3" H 10050 9899 50  0000 L CNN
-F 1 "MountingHole_Pad" H 10050 9808 50  0000 L CNN
+F 1 "DNI" H 10050 9808 50  0001 L CNN
 F 2 "MountingHole:MountingHole_2.2mm_M2_Pad_Via" H 9950 9850 50  0001 C CNN
 F 3 "~" H 9950 9850 50  0001 C CNN
@@
 F 2 "Package_TO_SOT_SMD:SOT-23-6" H 2800 9050 50  0001 L CIN
 F 3 "http://www.ti.com/lit/ds/symlink/tlv61046a.pdf" H 2750 9300 50  0001 C CNN
+F 4 "TLV61046ADBV" H 2750 9200 50  0001 C CNN "MPN"
+F 5 "3007283" H 2750 9200 50  0001 C CNN "Farnell"
 	1    2750 9200
 	1    0    0    -1
@@
 P 9950 10400
 F 0 "H4" H 10050 10449 50  0000 L CNN
-F 1 "MountingHole_Pad" H 10050 10358 50  0000 L CNN
+F 1 "DNI" H 10050 10358 50  0001 L CNN
 F 2 "MountingHole:MountingHole_2.2mm_M2_Pad_Via" H 9950 10400 50  0001 C CNN
 F 3 "~" H 9950 10400 50  0001 C CNN
@@
 F 2 "Package_SO:TSSOP-8_3x3mm_P0.65mm" H 3200 3400 50  0001 C CNN
 F 3 "http://www.ti.com/lit/sg/scyt129e/scyt129e.pdf" H 3200 3400 50  0001 C CNN
+F 4 "SN74LVC3G17DCT" H 3200 3400 50  0001 C CNN "MPN"
+F 5 "1236391" H 3200 3400 50  0001 C CNN "Farnell"
 	3    3200 3400
 	1    0    0    -1
@@
 F 2 "Connector_PinSocket_2.54mm:PinSocket_1x04_P2.54mm_Vertical" H 9750 7850 50  0001 C CNN
 F 3 "~" H 9750 7850 50  0001 C CNN
+F 4 "1593460" H 9750 7850 50  0001 C CNN "Farnell"
 	1    9750 7850
 	-1   0    0    1
@@
 P 9300 9550
 F 0 "MB1" H 9400 9550 50  0000 L CNN
-F 1 "MouseBite" H 9400 9505 50  0001 L CNN
+F 1 "DNI" H 9400 9505 50  0001 L CNN
 F 2 "Jitter_Footprints:MouseBite_3.5mmx2.2mm_breakaway" H 9300 9550 50  0001 C CNN
 F 3 "~" H 9300 9550 50  0001 C CNN
@@
 P 9300 9750
 F 0 "MB2" H 9400 9750 50  0000 L CNN
-F 1 "MouseBite" H 9400 9705 50  0001 L CNN
+F 1 "DNI" H 9400 9705 50  0001 L CNN
 F 2 "Jitter_Footprints:MouseBite_3.5mmx2.2mm_breakaway" H 9300 9750 50  0001 C CNN
 F 3 "~" H 9300 9750 50  0001 C CNN
@@
 P 9300 9950
 F 0 "MB3" H 9400 9950 50  0000 L CNN
-F 1 "MouseBite" H 9400 9905 50  0001 L CNN
+F 1 "DNI" H 9400 9905 50  0001 L CNN
 F 2 "Jitter_Footprints:MouseBite_3.5mmx2.2mm_breakaway" H 9300 9950 50  0001 C CNN
 F 3 "~" H 9300 9950 50  0001 C CNN
@@
 P 9300 10150
 F 0 "MB4" H 9400 10150 50  0000 L CNN
-F 1 "MouseBite" H 9400 10105 50  0001 L CNN
+F 1 "DNI" H 9400 10105 50  0001 L CNN
 F 2 "Jitter_Footprints:MouseBite_3.5mmx2.2mm_breakaway" H 9300 10150 50  0001 C CNN
 F 3 "~" H 9300 10150 50  0001 C CNN
@@
 P 8850 9750
 F 0 "TH2" H 8950 9750 50  0000 L CNN
-F 1 "ToolingHole" H 8950 9705 50  0001 L CNN
+F 1 "DNI" H 8950 9705 50  0001 L CNN
 F 2 "Jitter_Footprints:Tooling_hole_4mm_4.04mm_paste" H 8850 9750 50  0001 C CNN
 F 3 "~" H 8850 9750 50  0001 C CNN
@@
 P 8850 9550
 F 0 "TH1" H 8950 9550 50  0000 L CNN
-F 1 "ToolingHole" H 8950 9505 50  0001 L CNN
+F 1 "DNI" H 8950 9505 50  0001 L CNN
 F 2 "Jitter_Footprints:Tooling_hole_4mm_4.04mm_paste" H 8850 9550 50  0001 C CNN
 F 3 "~" H 8850 9550 50  0001 C CNN
@@
 P 8850 9950
 F 0 "TH3" H 8950 9950 50  0000 L CNN
-F 1 "ToolingHole" H 8950 9905 50  0001 L CNN
+F 1 "DNI" H 8950 9905 50  0001 L CNN
 F 2 "Jitter_Footprints:Tooling_hole_4mm_4.04mm_paste" H 8850 9950 50  0001 C CNN
 F 3 "~" H 8850 9950 50  0001 C CNN
@@
 P 8850 10150
 F 0 "TH4" H 8950 10150 50  0000 L CNN
-F 1 "ToolingHole" H 8950 10105 50  0001 L CNN
+F 1 "DNI" H 8950 10105 50  0001 L CNN
 F 2 "Jitter_Footprints:Tooling_hole_4mm_4.04mm_paste" H 8850 10150 50  0001 C CNN
 F 3 "~" H 8850 10150 50  0001 C CNN
@@
 	1    0    0    -1
 $EndComp
+Text Notes 1400 5600 0    50   ~ 0
+TODO all 10k resistors\nsame footprint!
 $EndSCHEMATC

Commit message: Fix BOM: add display as separate item
Parts:
- H1: Farnell (none) -> 3215747; MPN ELW2106AA -> 503480-1400; Mouser 387-ELW2106AA -> (none); Note (none) -> Requires a Futaba ELW2106AA display module
Changed lines of the file:
@@
 F 2 "Jitter_Footprints:Molex_503480-1400-1x14-1MP_P0.5mm_Horizontal" H 14200 3350 50  0001 C CNN
 F 3 "https://nl.mouser.com/datasheet/2/921/Futaba-10-02-2018-ELW2106AA_A_03_SHORT-1487521.pdf" H 14200 3350 50  0001 C CNN
-F 4 "ELW2106AA" H 14200 3350 50  0001 C CNN "MPN"
-F 5 "387-ELW2106AA" H 14200 3350 50  0001 C CNN "Mouser"
+F 4 "503480-1400" H 14200 3350 50  0001 C CNN "MPN"
+F 5 "3215747" H 14200 3350 50  0001 C CNN "Farnell"
+F 6 "Requires a Futaba ELW2106AA display module" H 14200 3350 50  0001 C CNN "Note"
 	1    14200 3350
 	1    0    0    -1
