File: pcb/serial-logger-prototype.sch (KiCad schematic (older format))
At the start: 69 parts, among them J1 JTAG/SWD, J2 Conn_01x04_Female, J3 Conn_01x04_Male, J4 Conn_01x03_Male, SW1 Rotary_Encoder_Switch_DualLED, SW2 SW_SPDT, U1 STM32G070KBT6, U2 74LVC3G17, U3 TLV70228_SOT23-5, U4 sn74lv1t34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

Commit message: Basic example of uart -> oled
However the uart interrupt is not handled fast enough causing overrun
errors. Even on optimize=2 with baudrate 9600. Next step is to implement
DMA to overcome this issue.
Other:
- note added: "Maybe we can connect this to a gpio pin \nso you can override it"
Changed lines of the file:
@@
 Text Notes 1400 5600 0    50   ~ 0
 TODO all 10k resistors\nsame footprint!
+Text Notes 8150 7200 0    50   ~ 0
+Maybe we can connect this to a gpio pin \nso you can override it
 $EndSCHEMATC

Commit message: Schematics: add note for next revision
Other:
- note added: "TODO check footprint:\nlooks like the pads are a bit far apart..?"
Changed lines of the file:
@@
 Text Notes 8150 7200 0    50   ~ 0
 Maybe we can connect this to a gpio pin \nso you can override it
+Text Notes 6800 8350 0    50   ~ 0
+TODO check footprint:\nlooks like the pads are a bit far apart..?
 $EndSCHEMATC
